Commit message: typo fix. Added gripper to urdf

File: urdf/phantomx_pincher_arm.xacro (robot description, xacro)
@@ -68,7 +68,7 @@
       </actuator>
     </transmission>
-  <!-- gripper
-  <xacro:include filename="$(find phantomx_pincher_arm_description)/urdf/phantomx_pincher_gripper.xacro"/> -->
-<!-- gripper_link
+  <!-- gripper -->
+  <xacro:include filename="phantomx_pincher_gripper.xacro"/>
+<!-- gripper_link -->
     <link name="gripper_link"/>
     <joint name="gripper_link_joint" type="revolute">
@@ -78,5 +78,5 @@
       <limit effort="6" velocity="1" lower="-3.14" upper="3.14"/>
       <axis xyz="1 0 0"/>
-    </joint> -->
+    </joint>
   <!--gazebo>
       <gripper name="gripper">
