Commit message: Added gripper controller

File: urdf/phantomx_pincher_gripper.xacro (robot description, xacro)
@@ -4,5 +4,5 @@
     <!-- gripper joint -->
     <!-- Finger 1 -->
-    <joint name="gripper_joint" type="prismatic">
+    <joint name="PhantomXPincher_gripperClose_joint" type="prismatic">
       <origin xyz="0.070 0 0" rpy="0 0 0"/>
       <axis xyz="0 1 0"/>

File: urdf/pincher_arm.urdf (robot description, URDF)
Before this commit: robot phantomx_pincher_arm, 7 links, 6 joints
Links:
- added link gripper_active2_link, mass 0.01; collision mesh filename=package://phantomx_pincher_arm_description/meshes/PincherFi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 scale=1.0 1.0 1.0; visual mesh filename=package://phantomx_pincher_arm_description/meshes/PincherFi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 scale=1.0 1.0 1.0
- added link gripper_active_link, mass 0.01; collision mesh filename=package://phantomx_pincher_arm_description/meshes/PincherFi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 scale=1.0 1.0 1.0; visual mesh filename=package://phantomx_pincher_arm_description/meshes/PincherFi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 scale=1.0 1.0 1.0
- link arm_base_link: mass None -> 0.055
- link arm_bicep_link: mass None -> 0.016
- link arm_forearm_link: mass None -> 0.016
- link arm_shoulder_pan_link: mass None -> 0.008
- link arm_wrist_flex_link: mass None -> 0.01
Joints:
- added joint PhantomXPincher_gripperClose_joint: type prismatic, parent arm_wrist_flex_link, child gripper_active_link, origin xyz=0.070 0 0 rpy=0 0 0, axis 0 1 0, limit lower=0.002 upper=0.032 effort=30 velocity=0.5
- added joint gripper2_joint: type fixed, parent arm_wrist_flex_link, child gripper_active2_link, origin xyz=0.070 -0.016 0 rpy=0 0 0
- joint PhantomXPincher_joint1: limit lower=-2.617 upper=2.617 effort=6 velocity=1.571 -> lower=-1.74 upper=1.74 effort=6 velocity=1.571
- joint PhantomXPincher_joint2: limit lower=-2.3 upper=2.3 effort=6 velocity=1.571 -> lower=-1.98 upper=1.88 effort=6 velocity=1.571
- joint PhantomXPincher_joint3: limit lower=-2.42 upper=2.38 effort=6 velocity=1.571 -> lower=-1.58 upper=0.59 effort=6 velocity=1.571
- joint PhantomXPincher_joint4: limit lower=-1.72 upper=1.68 effort=6 velocity=1.571 -> lower=-1.79 upper=1.67 effort=6 velocity=1.571
- joint arm_base_joint: origin xyz=0 0 0.020 rpy=0 0 0 -> xyz=0.0 0.00 0.077
