Commit message: corrected kinect cloud orientation

File: urdf/turtlebot2i.xacro (robot description, xacro)
@@ -3,256 +3,255 @@
   <xacro:property name="M_PI" value="3.1415926535897931" />
   <!-- Orbecc Astra Sensor -->
-    <joint name="camera1_joint" type="fixed">
-      <origin xyz="-0.088 0 0.225" rpy="${M_PI/2} 0 ${M_PI/2}"/>
-      <parent link="base_link"/>
-      <child link="camera1_link"/>
-    </joint>
-    <link name="camera1_link">
-      <visual>
-       <origin xyz="0 0 0" rpy="0 0 ${M_PI/2} "/>
-        <geometry>
-         <mesh filename="package://turtlebot_description/meshes/sensors/kinect.dae"/>
-        </geometry>
-      </visual>
-      <collision>
-        <origin xyz="0.0 0.0 0.0" rpy="0 0 0"/>
-        <geometry>
-          <box size="0.07271 0.27794 0.073"/>
-        </geometry>
-      </collision>
-      <inertial>
-        <mass value="0.564" />
-        <origin xyz="0 0 0" />
-        <inertia ixx="0.003881243" ixy="0.0" ixz="0.0"
-                 iyy="0.000498940" iyz="0.0"
-                 izz="0.003879257" />
-      </inertial>
-    </link>
+  <joint name="camera1_joint" type="fixed">
+    <origin xyz="-0.088 0 0.225" rpy="${-M_PI/2} 0 ${-M_PI/2}"/>
+    <parent link="base_link"/>
+    <child link="camera1_link_optical"/>
+  </joint>
+  <link name="camera1_link_optical">
+    <visual>
+      <origin xyz="0 0 0" rpy="${-M_PI/2} 0 ${M_PI}"/>
+      <geometry>
+       <mesh filename="package://turtlebot_description/meshes/sensors/kinect.dae"/>
+      </geometry>
+    </visual>
+    <collision>
+      <origin xyz="0.0 0.0 0.0" rpy="0 0 0"/>
+      <geometry>
+        <box size="0.07271 0.27794 0.073"/>
+      </geometry>
+    </collision>
+    <inertial>
+      <mass value="0.564" />
+      <origin xyz="0 0 0" />
+      <inertia ixx="0.003881243" ixy="0.0" ixz="0.0"
+               iyy="0.000498940" iyz="0.0"
+               izz="0.003879257" />
+    </inertial>
+  </link>
   <!-- Intel RealSense Sensor -->
-    <joint name="camera2_joint" type="fixed">
-      <origin xyz="0.112 0 0.4" rpy="0 1.05 0"/>
-      <parent link="base_link"/>
-      <child link="camera2_link"/>
-    </joint>
-    <link name="camera2_link">
-      <visual>
-       <origin xyz="0 0 0" rpy="0 0 0"/>
-        <geometry>
-         <mesh filename="package://turtlebot_description/meshes/sensors/kinect.dae"/>
-        </geometry>
-      </visual>
-      <collision>
-        <origin xyz="0.0 0.0 0.0" rpy="0 0 0"/>
-        <geometry>
-          <box size="0.07271 0.27794 0.073"/>
-        </geometry>
-      </collision>
-      <inertial>
-        <mass value="0.564" />
-        <origin xyz="0 0 0" />
-        <inertia ixx="0.003881243" ixy="0.0" ixz="0.0"
-                 iyy="0.000498940" iyz="0.0"
-                 izz="0.003879257" />
-      </inertial>
-    </link>
+  <joint name="camera2_joint" type="fixed">
+    <!--<origin xyz="0.112 0 0.4" rpy="1.05 0 ${M_PI/2}"/>-->
+    <origin xyz="0.112 0 0.4" rpy="0 0 0"/>
+    <parent link="base_link"/>
+    <child link="camera2_link"/>
+  </joint>
+  <link name="camera2_link">
+    <visual>
+     <origin xyz="0 0 0" rpy="1.05 0 ${M_PI/2}"/>
+      <geometry>
+       <mesh filename="package://turtlebot_description/meshes/sensors/kinect.dae"/>
+      </geometry>
+    </visual>
+    <collision>
+      <origin xyz="0.0 0.0 0.0" rpy="0 0 0"/>
+      <geometry>
+        <box size="0.07271 0.27794 0.073"/>
+      </geometry>
+    </collision>
+    <inertial>
+      <mass value="0.564" />
+      <origin xyz="0 0 0" />
+      <inertia ixx="0.003881243" ixy="0.0" ixz="0.0"
+               iyy="0.000498940" iyz="0.0"
+               izz="0.003879257" />
+    </inertial>
+  </link>
   <!-- Kobuki -->
-    <link name="base_footprint"/>
-    <!--
-       Base link is set at the bottom of the base mould.
-       This is done to be compatible with the way base link
-       was configured for turtlebot 1. Refer to
-       https://github.com/turtlebot/turtlebot/issues/40
-       To put the base link at the more oft used wheel
-       axis, set the z-distance from the base_footprint
-       to 0.352.
-      -->
-    <joint name="base_joint" type="fixed">
-      <origin xyz="0 0 0.0102" rpy="0 0 0" />
-      <parent link="base_footprint"/>
-      <child link="base_link" />
-    </joint>
-    <link name="base_link">
-      <visual>
-        <geometry>
-          <!-- new mesh -->
-          <mesh filename="package://kobuki_description/meshes/main_body.dae" />
-        </geometry>
-        <origin xyz="0.001 0 0.05199" rpy="0 0 0"/>
-      </visual>
-      <collision>
-        <geometry>
-          <cylinder length="0.10938" radius="0.178"/>
-        </geometry>
-        <origin xyz="0.0 0 0.05949" rpy="0 0 0"/>
-      </collision>
-      <inertial>
-        <!-- COM experimentally determined -->
-        <origin xyz="0.01 0 0"/>
-        <mass value="2.4"/> <!-- 2.4/2.6 kg for small/big battery pack -->
-        <!-- Kobuki's inertia tensor is approximated by a cylinder with homogeneous mass distribution
-             More details: http://en.wikipedia.org/wiki/List_of_moment_of_inertia_tensors
-             m = 2.4 kg; h = 0.09 m; r = 0.175 m
-             ixx = 1/12 * m * (3 * r^2 + h^2)
-             iyy = 1/12 * m * (3 * r^2 + h^2)
-             izz = 1/2 * m * r^2
-          -->
-        <inertia ixx="0.019995" ixy="0.0" ixz="0.0"
-                 iyy="0.019995" iyz="0.0"
-                 izz="0.03675" />
-      </inertial>
-    </link>
-    <joint name="wheel_left_joint" type="continuous">
-      <parent link="base_link"/>
-      <child link="wheel_left_link"/>
-      <origin xyz="0.00 ${0.23/2} 0.0250" rpy="${-M_PI/2} 0 0"/>
-      <axis xyz="0 0 1"/>
-    </joint>
-    <link name="wheel_left_link">
-      <visual>
-        <geometry>
-          <mesh filename="package://kobuki_description/meshes/wheel.dae"/>
-        </geometry>
-        <origin xyz="0 0 0" rpy="0 0 0"/>
-      </visual>
-      <collision>
-        <geometry>
-          <cylinder length="0.0206" radius="0.0352"/>
-        </geometry>
-        <origin rpy="0 0 0" xyz="0 0 0"/>
-      </collision>
-      <inertial>
-        <mass value="0.01" />
-        <origin xyz="0 0 0" />
-        <inertia ixx="0.001" ixy="0.0" ixz="0.0"
-                 iyy="0.001" iyz="0.0"
-                 izz="0.001" />
-      </inertial>
-    </link>
-    <joint name="wheel_right_joint" type="continuous">
-      <parent link="base_link"/>
-      <child link="wheel_right_link"/>
-      <origin xyz="0.00 -${0.23/2} 0.0250" rpy="${-M_PI/2} 0 0"/>
-      <axis xyz="0 0 1"/>
-    </joint>
-    <link name="wheel_right_link">
-      <visual>
-        <geometry>
-          <mesh filename="package://kobuki_description/meshes/wheel.dae"/>
-        </geometry>
-        <origin xyz="0 0 0" rpy="0 0 0"/>
-      </visual>
-      <collision>
-        <geometry>
-          <cylinder length="0.0206" radius="0.0350"/>
-        </geometry>
-        <origin rpy="0 0 0" xyz="0 0 0"/>
-      </collision>
-      <inertial>
-        <mass value="0.01" />
-        <origin xyz="0 0 0" />
-        <inertia ixx="0.001" ixy="0.0" ixz="0.0"
-                 iyy="0.001" iyz="0.0"
-                 izz="0.001" />
-      </inertial>
-    </link>
-    <joint name="caster_front_joint" type="fixed">
-      <parent link="base_link"/>
-      <child link="caster_front_link"/>
-      <origin xyz="0.115 0.0 0.007" rpy="${-M_PI/2} 0 0"/>
-    </joint>
-    <link name="caster_front_link">
-      <collision>
-        <geometry>
-          <cylinder length="0.0176" radius="0.017"/>
-        </geometry>
-        <origin rpy="0 0 0" xyz="0 0 0"/>
-      </collision>
-      <inertial>
-        <mass value="0.01" />
-        <origin xyz="0 0 0" />
-        <inertia ixx="0.001" ixy="0.0" ixz="0.0"
-                 iyy="0.001" iyz="0.0"
-                 izz="0.001" />
-      </inertial>
-    </link>
-    <joint name="caster_back_joint" type="fixed">
-      <parent link="base_link"/>
-      <child link="caster_back_link"/>
-      <origin xyz="-0.135 0.0 0.009" rpy="${-M_PI/2} 0 0"/>
-    </joint>
-    <link name="caster_back_link">
-      <collision>
-        <geometry>
-          <cylinder length="0.0176" radius="0.017"/>
-        </geometry>
-        <origin rpy="0 0 0" xyz="0 0 0"/>
-      </collision>
-      <inertial>
-        <mass value="0.01" />
-        <origin xyz="0 0 0" />
-        <inertia ixx="0.001" ixy="0.0" ixz="0.0"
-                 iyy="0.001" iyz="0.0"
-                 izz="0.001" />
-      </inertial>
-    </link>
-    <!-- Kobuki's sensors -->
-    <joint name="gyro_joint" type="fixed">
-      <axis xyz="0 1 0"/>
-      <origin xyz="0.056 0.062 0.0202" rpy="0 0 0"/>
-      <parent link="base_link"/>
-      <child link="gyro_link"/>
-    </joint>
-    <link name="gyro_link">
-      <inertial>
-        <mass value="0.001"/>
-        <origin xyz="0 0 0" rpy="0 0 0"/>
-        <inertia ixx="0.0001" ixy="0" ixz="0"
-                 iyy="0.000001" iyz="0"
-                 izz="0.0001"/>
-      </inertial>
-    </link>
-    <joint name="cliff_sensor_left_joint" type="fixed">
-      <origin xyz="0.08734 0.13601 0.0214" rpy="0 ${M_PI/2} 0" />
-      <parent link="base_link"/>
-      <child link="cliff_sensor_left_link" />
-    </joint>
-    <link name="cliff_sensor_left_link">
-      <inertial>
-        <mass value="0.0001" />
-        <origin xyz="0 0 0" />
-        <inertia ixx="0.0001" ixy="0.0" ixz="0.0"
-                 iyy="0.0001" iyz="0.0"
-                 izz="0.0001" />
-      </inertial>
-    </link>
-    <joint name="cliff_sensor_right_joint" type="fixed">
-      <origin xyz="0.085 -0.13601 0.0214" rpy="0 ${M_PI/2} 0" />
-      <parent link="base_link"/>
-      <child link="cliff_sensor_right_link" />
-    </joint>
-    <link name="cliff_sensor_right_link">
-      <inertial>
-        <mass value="0.0001" />
-        <origin xyz="0 0 0" />
-        <inertia ixx="0.0001" ixy="0.0" ixz="0.0"
-                 iyy="0.0001" iyz="0.0"
-                 izz="0.0001" />
-      </inertial>
-    </link>
-    <joint name="cliff_sensor_front_joint" type="fixed">
-      <origin xyz="0.156 0.00 0.0214" rpy="0 ${M_PI/2} 0" />
-      <parent link="base_link"/>
-      <child link="cliff_sensor_front_link" />
-    </joint>
-    <link name="cliff_sensor_front_link">
-      <inertial>
-        <mass value="0.0001" />
-        <origin xyz="0 0 0" />
-        <inertia ixx="0.0001" ixy="0.0" ixz="0.0"
-                 iyy="0.0001" iyz="0.0"
-                 izz="0.0001" />
-      </inertial>
-    </link>
-    <!-- Kobuki Gazebo simulation details -->
-    <!--<kobuki_sim_crumb/>-->
+  <link name="base_footprint"/>
+  <!--
+     Base link is set at the bottom of the base mould.
+     This is done to be compatible with the way base link
+     was configured for turtlebot 1. Refer to
+     https://github.com/turtlebot/turtlebot/issues/40
+     To put the base link at the more oft used wheel
+     axis, set the z-distance from the base_footprint
+     to 0.352.
+    -->
+  <joint name="base_joint" type="fixed">
+    <origin xyz="0 0 0.0102" rpy="0 0 0" />
+    <parent link="base_footprint"/>
+    <child link="base_link" />
+  </joint>
+  <link name="base_link">
+    <visual>
+      <geometry>
+        <!-- new mesh -->
+        <mesh filename="package://kobuki_description/meshes/main_body.dae" />
+      </geometry>
+      <origin xyz="0.001 0 0.05199" rpy="0 0 0"/>
+    </visual>
+    <collision>
+      <geometry>
+        <cylinder length="0.10938" radius="0.178"/>
+      </geometry>
+      <origin xyz="0.0 0 0.05949" rpy="0 0 0"/>
+    </collision>
+    <inertial>
+      <!-- COM experimentally determined -->
+      <origin xyz="0.01 0 0"/>
+      <mass value="2.4"/> <!-- 2.4/2.6 kg for small/big battery pack -->
+      <!-- Kobuki's inertia tensor is approximated by a cylinder with homogeneous mass distribution
+           More details: http://en.wikipedia.org/wiki/List_of_moment_of_inertia_tensors
+           m = 2.4 kg; h = 0.09 m; r = 0.175 m
+           ixx = 1/12 * m * (3 * r^2 + h^2)
+           iyy = 1/12 * m * (3 * r^2 + h^2)
+           izz = 1/2 * m * r^2
+        -->
+      <inertia ixx="0.019995" ixy="0.0" ixz="0.0"
+               iyy="0.019995" iyz="0.0"
+               izz="0.03675" />
+    </inertial>
+  </link>
+  <joint name="wheel_left_joint" type="continuous">
+    <parent link="base_link"/>
+    <child link="wheel_left_link"/>
+    <origin xyz="0.00 ${0.23/2} 0.0250" rpy="${-M_PI/2} 0 0"/>
+    <axis xyz="0 0 1"/>
+  </joint>
+  <link name="wheel_left_link">
+    <visual>
+      <geometry>
+        <mesh filename="package://kobuki_description/meshes/wheel.dae"/>
+      </geometry>
+      <origin xyz="0 0 0" rpy="0 0 0"/>
+    </visual>
+    <collision>
+      <geometry>
+        <cylinder length="0.0206" radius="0.0352"/>
+      </geometry>
+      <origin rpy="0 0 0" xyz="0 0 0"/>
+    </collision>
+    <inertial>
+      <mass value="0.01" />
+      <origin xyz="0 0 0" />
+      <inertia ixx="0.001" ixy="0.0" ixz="0.0"
+               iyy="0.001" iyz="0.0"
+               izz="0.001" />
+    </inertial>
+  </link>
+  <joint name="wheel_right_joint" type="continuous">
+    <parent link="base_link"/>
+    <child link="wheel_right_link"/>
+    <origin xyz="0.00 -${0.23/2} 0.0250" rpy="${-M_PI/2} 0 0"/>
+    <axis xyz="0 0 1"/>
+  </joint>
+  <link name="wheel_right_link">
+    <visual>
+      <geometry>
+        <mesh filename="package://kobuki_description/meshes/wheel.dae"/>
+      </geometry>
+      <origin xyz="0 0 0" rpy="0 0 0"/>
+    </visual>
+    <collision>
+      <geometry>
+        <cylinder length="0.0206" radius="0.0350"/>
+      </geometry>
+      <origin rpy="0 0 0" xyz="0 0 0"/>
+    </collision>
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
Commit message: fixed point cloud output from active camera

File: urdf/turtlebot2i.xacro (robot description, xacro)
@@ -4,11 +4,12 @@
   <!-- Orbecc Astra Sensor -->
   <joint name="camera1_joint" type="fixed">
-    <origin xyz="-0.088 0 0.225" rpy="${-M_PI/2} 0 ${-M_PI/2}"/>
-    <parent link="base_link"/>
-    <child link="camera1_link_optical"/>
-  </joint>
-  <link name="camera1_link_optical">
-    <visual>
-      <origin xyz="0 0 0" rpy="${-M_PI/2} 0 ${M_PI}"/>
+    <origin xyz="-0.088 0 0.28" rpy="${M_PI/2} 0 ${M_PI/2}"/>
+    <!--<origin xyz="-0.088 0 0.225" rpy="${M_PI/2} 0 ${M_PI/2}"/>-->
+    <parent link="base_link"/>
+    <child link="camera1_link"/>
+  </joint>
+  <link name="camera1_link">
+    <visual>
+      <origin xyz="0 0 0" rpy="${-M_PI/2} 0 0"/>
       <geometry>
        <mesh filename="package://turtlebot_description/meshes/sensors/kinect.dae"/>
@@ -31,6 +32,6 @@
   <!-- Intel RealSense Sensor -->
   <joint name="camera2_joint" type="fixed">
-    <!--<origin xyz="0.112 0 0.4" rpy="1.05 0 ${M_PI/2}"/>-->
-    <origin xyz="0.112 0 0.4" rpy="0 0 0"/>
+    <origin xyz="0.112 -0.025 0.454" rpy="${M_PI/3+M_PI/2} 0 ${M_PI/2}"/>
+    <!--<origin xyz="0.112 0 0.4" rpy="${M_PI/3+M_PI/2} 0 ${M_PI/2}"/>-->
     <parent link="base_link"/>
     <child link="camera2_link"/>
@@ -38,5 +39,6 @@
   <link name="camera2_link">
     <visual>
-     <origin xyz="0 0 0" rpy="1.05 0 ${M_PI/2}"/>
+     <!--<origin xyz="0 0 0" rpy="1.05 0 ${M_PI/2}"/>-->
+     <origin xyz="0 0 0" rpy="${-M_PI/2} 0 0"/>
       <geometry>
        <mesh filename="package://turtlebot_description/meshes/sensors/kinect.dae"/>

Commit message: fixed some point cloud issues

File: urdf/turtlebot2i.xacro (robot description, xacro)
@@ -4,5 +4,6 @@
   <!-- Orbecc Astra Sensor -->
   <joint name="camera1_joint" type="fixed">
-    <origin xyz="-0.088 0 0.28" rpy="${M_PI/2} 0 ${M_PI/2}"/>
+    <origin xyz="-0.088 0 0.32" rpy="${M_PI/2} 0 ${M_PI/2}"/>
+    <!--<origin xyz="-0.088 0 0.28" rpy="${M_PI/2} 0 ${M_PI/2}"/>-->
     <!--<origin xyz="-0.088 0 0.225" rpy="${M_PI/2} 0 ${M_PI/2}"/>-->
     <parent link="base_link"/>
@@ -32,4 +33,5 @@
   <!-- Intel RealSense Sensor -->
   <joint name="camera2_joint" type="fixed">
+    <!--<origin xyz="0.112 -0.025 0.454" rpy="0 0 0"/>-->
     <origin xyz="0.112 -0.025 0.454" rpy="${M_PI/3+M_PI/2} 0 ${M_PI/2}"/>
     <!--<origin xyz="0.112 0 0.4" rpy="${M_PI/3+M_PI/2} 0 ${M_PI/2}"/>-->

Commit message: script loaded by robot name, fixed robot tf, fixed lidar returns and added a new scenario

File: urdf/turtlebot2i.xacro (robot description, xacro)
@@ -2,4 +2,32 @@
 <robot name="turtlebot2i" xmlns:xacro="http://ros.org/wiki/xacro">
   <xacro:property name="M_PI" value="3.1415926535897931" />
+  <!-- Hokuyo LiDAR Sensor -->
+  <joint name="lidar_joint" type="fixed">
+    <origin xyz="0 0 0.485" rpy="0 0 0"/>
+    <parent link="base_link"/>
+    <child link="scan"/>
+  </joint>
+  <link name="scan">
+    <visual>
+      <origin xyz="0 0 0" rpy="0 0 0"/>
+      <geometry>
+       <!--<mesh filename="package://turtlebot_description/meshes/sensors/kinect.dae"/>-->
+        <box size="0.08 0.08 0.08"/>
+      </geometry>
+    </visual>
+    <collision>
+      <origin xyz="0.0 0.0 0.0" rpy="0 0 0"/>
+      <geometry>
+        <box size="0.08 0.08 0.08"/>
+      </geometry>
+    </collision>
+    <inertial>
+      <mass value="0.564" />
+      <origin xyz="0 0 0" />
+      <inertia ixx="0.003881243" ixy="0.0" ixz="0.0"
+               iyy="0.000498940" iyz="0.0"
+               izz="0.003879257" />
+    </inertial>
+  </link>
   <!-- Orbecc Astra Sensor -->
   <joint name="camera1_joint" type="fixed">
