Commit message: fixing urdf/movit integration error

File: src/phantomx_pincher_arm/phantomx_pincher_arm_description/urdf/phantomx_pincher_arm.urdf.xacro (robot description, xacro)
@@ -5,12 +5,12 @@
     to allow access to different operational areas, e.g. left handed vs. right handed robot -->
     <xacro:property name="joints_vlimit" value="1.571"/>
-    <xacro:property name="pan_llimit" value="-3.14"/>
-    <xacro:property name="pan_ulimit" value="3.14"/>
-    <xacro:property name="shoulder_llimit" value="-3.14"/>
-    <xacro:property name="shoulder_ulimit" value="3.14"/>
-    <xacro:property name="elbow_llimit" value="-3.14"/>
-    <xacro:property name="elbow_ulimit" value="3.14"/>
-    <xacro:property name="wrist_llimit" value="-3.14"/>
-    <xacro:property name="wrist_ulimit" value="3.14"/>
+    <xacro:property name="pan_llimit" value="-1.74"/>
+    <xacro:property name="pan_ulimit" value="1.74"/>
+    <xacro:property name="shoulder_llimit" value="-1.98"/>
+    <xacro:property name="shoulder_ulimit" value="1.88"/>
+    <xacro:property name="elbow_llimit" value="-1.58"/>
+    <xacro:property name="elbow_ulimit" value="1.59"/>
+    <xacro:property name="wrist_llimit" value="-1.79"/>
+    <xacro:property name="wrist_ulimit" value="1.67"/>
     <!-- Included URDF Files -->
     <xacro:include filename="phantomx_pincher_arm.xacro"/>

File: src/phantomx_pincher_arm/phantomx_pincher_arm_description/urdf/phantomx_pincher_arm.xacro (robot description, xacro)
@@ -69,5 +69,5 @@
     </transmission>
   <!-- gripper -->
-  <xacro:include filename="phantomx_pincher_gripper.xacro"/>
+  <xacro:include filename="$(find phantomx_pincher_arm_description)/urdf/phantomx_pincher_gripper.xacro"/>
 <!-- gripper_link -->
     <link name="gripper_link"/>

File: src/turtlebot2i/turtlebot2i_description/urdf/arms/phantomx_pincher_arm.urdf.xacro (robot description, xacro)
@@ -5,12 +5,12 @@
     to allow access to different operational areas, e.g. left handed vs. right handed robot -->
     <xacro:property name="joints_vlimit" value="1.571"/>
-    <xacro:property name="pan_llimit" value="-3.14"/>
-    <xacro:property name="pan_ulimit" value="3.14"/>
-    <xacro:property name="shoulder_llimit" value="-3.14"/>
-    <xacro:property name="shoulder_ulimit" value="3.14"/>
-    <xacro:property name="elbow_llimit" value="-3.14"/>
-    <xacro:property name="elbow_ulimit" value="3.14"/>
-    <xacro:property name="wrist_llimit" value="-3.14"/>
-    <xacro:property name="wrist_ulimit" value="3.14"/>
+    <xacro:property name="pan_llimit" value="-1.74"/>
+    <xacro:property name="pan_ulimit" value="1.74"/>
+    <xacro:property name="shoulder_llimit" value="-1.98"/>
+    <xacro:property name="shoulder_ulimit" value="1.88"/>
+    <xacro:property name="elbow_llimit" value="-1.58"/>
+    <xacro:property name="elbow_ulimit" value="1.59"/>
+    <xacro:property name="wrist_llimit" value="-1.79"/>
+    <xacro:property name="wrist_ulimit" value="1.67"/>
     <!-- We can configure joints velocity limit and lower/upper limits
     to allow access to different operational areas, e.g. left handed vs. right handed robot -->
