Commit message: Making files more generic. But still need improvement

File: phantomx_pincher_arm_description/urdf/arm_hardware.xacro (robot description, xacro)
@@ -56,14 +56,14 @@
       </inertial>
       <visual>
+        <origin xyz="-0.115 0 -0.2" rpy="0 0 0"/>
+        <geometry>
+          <mesh filename="package://phantomx_pincher_arm_description/meshes/PincherMotor.stl" scale="1.0 1.0 1.0"/>
+        </geometry>
+        <material name="${color}"/>
+      </visual>
+      <collision>
         <origin xyz="0 0 0" rpy="0 0 0"/>
         <geometry>
-          <mesh filename="package://phantomx_pincher_arm_description/meshes/F2Bracket.stl" scale="1.0 1.0 1.0"/>
-        </geometry>
-        <material name="${color}"/>
-      </visual>
-      <collision>
-        <origin xyz="0 0 0" rpy="0 0 0"/>
-        <geometry>
-          <mesh filename="package://phantomx_pincher_arm_description/meshes/F2Bracket.stl" scale="1.0 1.0 1.0"/>
+          <mesh filename="package://phantomx_pincher_arm_description/meshes/PincherMotor.stl" scale="1.0 1.0 1.0"/>
         </geometry>
       </collision>
@@ -93,7 +93,7 @@
       </inertial>
       <visual>
-        <origin xyz=" 0 0 0 " rpy="0 0 0"/>
-        <geometry>
-          <mesh filename="package://phantomx_pincher_arm_description/meshes/PincherBicep.stl" scale="1.0 1.0 1.0"/>
+        <origin xyz=" 0 0 0 " rpy="0 -1.54 0"/>
+        <geometry>
+          <mesh filename="package://phantomx_pincher_arm_description/meshes/PincherForeArm.stl" scale="1.0 1.0 1.0"/>
         </geometry>
         <material name="${color}"/>
@@ -102,5 +102,5 @@
         <origin xyz="0.0 0.0 0.0" rpy="0 0 0"/>
         <geometry>
-          <mesh filename="package://phantomx_pincher_arm_description/meshes/PincherBicep.stl" scale="1.0 1.0 1.0"/>
+          <mesh filename="package://phantomx_pincher_arm_description/meshes/PincherForeArm.stl" scale="1.0 1.0 1.0"/>
         </geometry>
       </collision>

File: phantomx_pincher_arm_description/urdf/phantomx_pincher_arm.xacro (robot description, xacro)
@@ -41,5 +41,5 @@
     <pincher_forearm parent="arm_bicep_link" name="arm_forearm" color="${color}"
                          vlimit="${joints_vlimit}" llimit="${elbow_llimit}" ulimit="${elbow_ulimit}">
-      <origin xyz="0.0325 0 0.104" rpy="0 0 0"/>
+      <origin xyz="0 0 0.104" rpy="3.14 -1.57 0"/>
     </pincher_forearm>
     <transmission name="arm_forearm_transmission">
@@ -72,5 +72,5 @@
 <!-- gripper_link -->
     <link name="gripper_link"/>
-    <joint name="gripper_link_joint" type="revolute">
+    <joint name="PhantomXPincher_gripperCenter_joint" type="revolute">
       <origin xyz="0.110 0 0" rpy="0 0 0"/>
       <parent link="arm_wrist_flex_link"/>

Commit message: Modification to control one of two robots on scene

File: phantomx_pincher_arm_description/urdf/arm_hardware.xacro (robot description, xacro)
@@ -38,5 +38,5 @@
   </xacro:macro>
   <xacro:macro name="bracket_F2_revolute" params="parent name color llimit ulimit vlimit *origin">
-    <joint name="PhantomXPincher_joint1" type="revolute">
+    <joint name="$(arg joint1)" type="revolute">
       <xacro:insert_block name="origin"/>
       <axis xyz="0 0 1"/>
@@ -75,5 +75,5 @@
   </xacro:macro>
   <xacro:macro name="pincher_bicep" params="parent name color llimit ulimit vlimit *origin">
-    <joint name="PhantomXPincher_joint2" type="revolute">
+    <joint name="$(arg joint2)" type="revolute">
       <xacro:insert_block name="origin"/>
       <axis xyz="0 1 0"/>
@@ -112,5 +112,5 @@
   </xacro:macro>
   <xacro:macro name="pincher_forearm" params="parent name color llimit ulimit vlimit *origin">
-    <joint name="PhantomXPincher_joint3" type="revolute">
+    <joint name="$(arg joint3)" type="revolute">
       <xacro:insert_block name="origin"/>
       <axis xyz="0 -1 0"/>
@@ -149,5 +149,5 @@
   </xacro:macro>
   <xacro:macro name="pincher_wrist" params="parent name color llimit ulimit vlimit *origin">
-    <joint name="PhantomXPincher_joint4" type="revolute">
+    <joint name="$(arg joint4)" type="revolute">
       <xacro:insert_block name="origin"/>
       <axis xyz="0 -1 0"/>

File: phantomx_pincher_arm_description/urdf/phantomx_pincher_arm.xacro (robot description, xacro)
@@ -15,5 +15,5 @@
     <transmission name="arm_shoulder_pan_transmission">
       <type>transmission_interface/SimpleTransmission</type>
-      <joint name="PhantomXPincher_joint1">
+      <joint name="$(arg joint1)">
         <hardwareInterface>EffortJointInterface</hardwareInterface>
       </joint>
@@ -30,5 +30,5 @@
     <transmission name="arm_bicep_transmission">
       <type>transmission_interface/SimpleTransmission</type>
-      <joint name="PhantomXPincher_joint2">
+      <joint name="$(arg joint2)">
         <hardwareInterface>EffortJointInterface</hardwareInterface>
       </joint>
@@ -45,5 +45,5 @@
     <transmission name="arm_forearm_transmission">
       <type>transmission_interface/SimpleTransmission</type>
-      <joint name="PhantomXPincher_joint3">
+      <joint name="$(arg joint3)">
         <hardwareInterface>EffortJointInterface</hardwareInterface>
       </joint>
@@ -60,5 +60,5 @@
     <transmission name="arm_wrist_flex_transmission">
       <type>transmission_interface/SimpleTransmission</type>
-      <joint name="PhantomXPincher_joint4">
+      <joint name="$(arg joint4)">
         <hardwareInterface>EffortJointInterface</hardwareInterface>
       </joint>
@@ -72,5 +72,5 @@
 <!-- gripper_link -->
     <link name="gripper_link"/>
-    <joint name="PhantomXPincher_gripperCenter_joint" type="revolute">
+    <joint name="$(arg gripper2)" type="revolute">
       <origin xyz="0.110 0 0" rpy="0 0 0"/>
       <parent link="arm_wrist_flex_link"/>

File: phantomx_pincher_arm_description/urdf/phantomx_pincher_gripper.xacro (robot description, xacro)
@@ -4,5 +4,5 @@
     <!-- gripper joint -->
     <!-- Finger 1 -->
-    <joint name="PhantomXPincher_gripperClose_joint" type="prismatic">
+    <joint name="$(arg gripper1)" type="prismatic">
       <origin xyz="0.070 0 0" rpy="0 0 0"/>
       <axis xyz="0 1 0"/>

Commit message: Making all joint names the same as on the standart robot.

File: phantomx_pincher_arm_description/urdf/arm_hardware.xacro (robot description, xacro)
@@ -38,5 +38,5 @@
   </xacro:macro>
   <xacro:macro name="bracket_F2_revolute" params="parent name color llimit ulimit vlimit *origin">
-    <joint name="$(arg joint1)" type="revolute">
+    <joint name="PhantomXPincher_joint1" type="revolute">
       <xacro:insert_block name="origin"/>
       <axis xyz="0 0 1"/>
@@ -75,5 +75,5 @@
   </xacro:macro>
   <xacro:macro name="pincher_bicep" params="parent name color llimit ulimit vlimit *origin">
-    <joint name="$(arg joint2)" type="revolute">
+    <joint name="PhantomXPincher_joint2" type="revolute">
       <xacro:insert_block name="origin"/>
       <axis xyz="0 1 0"/>
@@ -112,5 +112,5 @@
   </xacro:macro>
   <xacro:macro name="pincher_forearm" params="parent name color llimit ulimit vlimit *origin">
-    <joint name="$(arg joint3)" type="revolute">
+    <joint name="PhantomXPincher_joint3" type="revolute">
       <xacro:insert_block name="origin"/>
       <axis xyz="0 -1 0"/>
@@ -149,5 +149,5 @@
   </xacro:macro>
   <xacro:macro name="pincher_wrist" params="parent name color llimit ulimit vlimit *origin">
-    <joint name="$(arg joint4)" type="revolute">
+    <joint name="PhantomXPincher_joint4" type="revolute">
       <xacro:insert_block name="origin"/>
       <axis xyz="0 -1 0"/>

File: phantomx_pincher_arm_description/urdf/phantomx_pincher_arm.xacro (robot description, xacro)
@@ -15,5 +15,5 @@
     <transmission name="arm_shoulder_pan_transmission">
       <type>transmission_interface/SimpleTransmission</type>
-      <joint name="$(arg joint1)">
+      <joint name="PhantomXPincher_joint1">
         <hardwareInterface>EffortJointInterface</hardwareInterface>
       </joint>
@@ -30,5 +30,5 @@
     <transmission name="arm_bicep_transmission">
       <type>transmission_interface/SimpleTransmission</type>
-      <joint name="$(arg joint2)">
+      <joint name="PhantomXPincher_joint2">
         <hardwareInterface>EffortJointInterface</hardwareInterface>
       </joint>
@@ -45,5 +45,5 @@
     <transmission name="arm_forearm_transmission">
       <type>transmission_interface/SimpleTransmission</type>
-      <joint name="$(arg joint3)">
+      <joint name="PhantomXPincher_joint3">
         <hardwareInterface>EffortJointInterface</hardwareInterface>
       </joint>
@@ -60,5 +60,5 @@
     <transmission name="arm_wrist_flex_transmission">
       <type>transmission_interface/SimpleTransmission</type>
-      <joint name="$(arg joint4)">
+      <joint name="PhantomXPincher_joint4">
         <hardwareInterface>EffortJointInterface</hardwareInterface>
       </joint>
@@ -72,5 +72,5 @@
 <!-- gripper_link -->
     <link name="gripper_link"/>
-    <joint name="$(arg gripper2)" type="revolute">
+    <joint name="PhantomXPincher_gripperCenter_joint" type="revolute">
       <origin xyz="0.110 0 0" rpy="0 0 0"/>
       <parent link="arm_wrist_flex_link"/>

File: phantomx_pincher_arm_description/urdf/phantomx_pincher_gripper.xacro (robot description, xacro)
@@ -4,5 +4,5 @@
     <!-- gripper joint -->
     <!-- Finger 1 -->
-    <joint name="$(arg gripper1)" type="prismatic">
+    <joint name="PhantomXPincher_gripperClose_joint" type="prismatic">
       <origin xyz="0.070 0 0" rpy="0 0 0"/>
       <axis xyz="0 1 0"/>

Commit message: Updated arm urdf to match the real arm

File: phantomx_pincher_arm_description/urdf/arm_hardware.xacro (robot description, xacro)
@@ -56,14 +56,14 @@
       </inertial>
       <visual>
-        <origin xyz="-0.115 0 -0.2" rpy="0 0 0"/>
-        <geometry>
-          <mesh filename="package://phantomx_pincher_arm_description/meshes/PincherMotor.stl" scale="1.0 1.0 1.0"/>
-        </geometry>
-        <material name="${color}"/>
-      </visual>
-      <collision>
-        <origin xyz="0 0 0" rpy="0 0 0"/>
-        <geometry>
-          <mesh filename="package://phantomx_pincher_arm_description/meshes/PincherMotor.stl" scale="1.0 1.0 1.0"/>
+        <origin xyz="0 0 0" rpy="0 0 0"/>
+        <geometry>
+          <mesh filename="package://phantomx_pincher_arm_description/meshes/F2Bracket.stl" scale="1.0 1.0 1.0"/>
+        </geometry>
+        <material name="${color}"/>
+      </visual>
+      <collision>
+        <origin xyz="0 0 0" rpy="0 0 0"/>
+        <geometry>
+          <mesh filename="package://phantomx_pincher_arm_description/meshes/F2Bracket.stl" scale="1.0 1.0 1.0"/>
         </geometry>
       </collision>
@@ -93,7 +93,7 @@
       </inertial>
       <visual>
-        <origin xyz=" 0 0 0 " rpy="0 -1.54 0"/>
-        <geometry>
-          <mesh filename="package://phantomx_pincher_arm_description/meshes/PincherForeArm.stl" scale="1.0 1.0 1.0"/>
+        <origin xyz=" 0 0 0 " rpy="0 0 0"/>
+        <geometry>
+          <mesh filename="package://phantomx_pincher_arm_description/meshes/PincherBicep.stl" scale="1.0 1.0 1.0"/>
         </geometry>
         <material name="${color}"/>
@@ -102,5 +102,5 @@
         <origin xyz="0.0 0.0 0.0" rpy="0 0 0"/>
         <geometry>
-          <mesh filename="package://phantomx_pincher_arm_description/meshes/PincherForeArm.stl" scale="1.0 1.0 1.0"/>
+          <mesh filename="package://phantomx_pincher_arm_description/meshes/PincherBicep.stl" scale="1.0 1.0 1.0"/>
         </geometry>
       </collision>
@@ -130,5 +130,5 @@
       </inertial>
       <visual>
-        <origin xyz=" 0 0 0 " rpy="0 0 0"/>
+        <origin xyz="0 0.0 0 " rpy="0 0 0"/>
         <geometry>
           <mesh filename="package://phantomx_pincher_arm_description/meshes/PincherForeArm.stl" scale="1.0 1.0 1.0"/>

File: phantomx_pincher_arm_description/urdf/phantomx_pincher_arm.xacro (robot description, xacro)
@@ -41,5 +41,5 @@
     <pincher_forearm parent="arm_bicep_link" name="arm_forearm" color="${color}"
                          vlimit="${joints_vlimit}" llimit="${elbow_llimit}" ulimit="${elbow_ulimit}">
-      <origin xyz="0 0 0.104" rpy="3.14 -1.57 0"/>
+      <origin xyz="0.0325 0 0.104" rpy="0 -1.57 0"/>
     </pincher_forearm>
     <transmission name="arm_forearm_transmission">
