Commit message: fixed camera frame and publishing

File: src/turtlebot2i/turtlebot2i_description/urdf/sensors/astra.urdf.xacro (robot description, xacro)
@@ -64,5 +64,6 @@
     <link name="camera_depth_frame"/>
     <joint name="camera_depth_optical_joint" type="fixed">
-      <origin xyz="0 0 0" rpy="${-M_PI/2} 0 ${-M_PI/2}" />
+      <!--<origin xyz="0 0 0" rpy="${-M_PI/2} 0 ${-M_PI/2}" />-->
+      <origin xyz="0 0 0" rpy="${-M_PI/2} ${M_PI} ${-M_PI/2}" />
       <parent link="camera_depth_frame" />
       <child link="camera_depth_optical_frame" />

File: src/turtlebot2i/turtlebot2i_description/urdf/sensors/sr300.urdf.xacro (robot description, xacro)
@@ -80,5 +80,5 @@
     <link name="camera_sr300_depth_frame"/>
     <joint name="camera_sr300_depth_optical_joint" type="fixed">
-        <origin xyz="0 0 0" rpy="${-M_PI/2} 0 ${-M_PI/2}" />
+        <origin xyz="0 0 0" rpy="${-M_PI/2-M_PI/26} ${M_PI} ${-M_PI/2}" />
         <parent link="camera_sr300_depth_frame" />
         <child link="camera_sr300_depth_optical_frame" />
