Commit message: Fix joint limits

File: src/turtlebot2i/turtlebot2i_description/urdf/arms/phantomx_pincher_arm.urdf.xacro (robot description, xacro)
@@ -5,12 +5,12 @@
     to allow access to different operational areas, e.g. left handed vs. right handed robot -->
     <xacro:property name="joints_vlimit" value="1.571"/>
-    <xacro:property name="pan_llimit" value="-1.74"/>
-    <xacro:property name="pan_ulimit" value="1.74"/>
-    <xacro:property name="shoulder_llimit" value="-1.98"/>
-    <xacro:property name="shoulder_ulimit" value="1.88"/>
-    <xacro:property name="elbow_llimit" value="-1.58"/>
-    <xacro:property name="elbow_ulimit" value="1.59"/>
-    <xacro:property name="wrist_llimit" value="-1.79"/>
-    <xacro:property name="wrist_ulimit" value="1.67"/>
+    <xacro:property name="pan_llimit" value="-3.1416"/>
+    <xacro:property name="pan_ulimit" value="3.1416"/>
+    <xacro:property name="shoulder_llimit" value="-1.83"/>
+    <xacro:property name="shoulder_ulimit" value="1.83"/>
+    <xacro:property name="elbow_llimit" value="-3.1416"/>
+    <xacro:property name="elbow_ulimit" value="0.33516"/>
+    <xacro:property name="wrist_llimit" value="-1.57"/>
+    <xacro:property name="wrist_ulimit" value="1.57"/>
     <!-- We can configure joints velocity limit and lower/upper limits
     to allow access to different operational areas, e.g. left handed vs. right handed robot -->

File: src/turtlebot2i/turtlebot2i_description/urdf/turtlebot_library.urdf.xacro (robot description, xacro)
@@ -17,4 +17,5 @@
   <xacro:include filename="$(find turtlebot2i_description)/urdf/sensors/scanse.urdf.xacro"/>
   <!-- Arms -->
-  <xacro:include filename="$(find turtlebot2i_description)/urdf/arms/phantomx_pincher_arm.urdf.xacro"/>
+ <!-- <xacro:include filename="$(find phantomx_pincher_arm_description)/urdf/phantomx_pincher_arm.urdf.xacro"/> -->
+ <xacro:include filename="$(find turtlebot2i_description)/urdf/arms/phantomx_pincher_arm.urdf.xacro"/>
 </robot>
