Commit message: robot description with integration of the base robot and arm

File: src/turtlebot2i/turtlebot2i_description/robots/kobuki_interbotix_astra.urdf.xacro (robot description, xacro)
@@ -13,5 +13,6 @@
   <sensor_sr300 parent="base_link"/>
   <phantomx_pincher_arm parent="base_link" color="Red" gripper_color="Red">
-    <origin xyz="0.145 0.0 0.112"/>
+    <!--<origin xyz="0.145 0.0 0.112"/>-->
+    <origin xyz="0.145 0.0 0.148"/>
   </phantomx_pincher_arm>
 </robot>

File: src/turtlebot2i/turtlebot2i_description/urdf/arms/phantomx_pincher_arm.urdf.xacro (robot description, xacro)
@@ -3,15 +3,17 @@
 <robot name="phantomx_pincher_arm" xmlns:xacro="http://ros.org/wiki/xacro">
     <!-- We can configure joints velocity limit and lower/upper limits
-          to allow access to different operational areas, e.g. left handed vs. right handed robot -->
+    to allow access to different operational areas, e.g. left handed vs. right handed robot -->
     <xacro:property name="joints_vlimit" value="1.571"/>
-    <xacro:property name="pan_llimit" value="-1.74"/>
-    <xacro:property name="pan_ulimit" value="1.74"/>
-    <xacro:property name="shoulder_llimit" value="-1.98"/>
-    <xacro:property name="shoulder_ulimit" value="1.88"/>
-    <xacro:property name="elbow_llimit" value="-1.58"/>
-    <xacro:property name="elbow_ulimit" value="0.59"/>
-    <xacro:property name="wrist_llimit" value="-1.79"/>
-    <xacro:property name="wrist_ulimit" value="1.67"/>
+    <xacro:property name="pan_llimit" value="-3.14"/>
+    <xacro:property name="pan_ulimit" value="3.14"/>
+    <xacro:property name="shoulder_llimit" value="-3.14"/>
+    <xacro:property name="shoulder_ulimit" value="3.14"/>
+    <xacro:property name="elbow_llimit" value="-3.14"/>
+    <xacro:property name="elbow_ulimit" value="3.14"/>
+    <xacro:property name="wrist_llimit" value="-3.14"/>
+    <xacro:property name="wrist_ulimit" value="3.14"/>
+    <!-- We can configure joints velocity limit and lower/upper limits
+    to allow access to different operational areas, e.g. left handed vs. right handed robot -->
     <!-- Included URDF Files -->
-    <xacro:include filename="$(find phantomx_pincher_arm_description)/urdf/phantomx_pincher_arm.xacro" />
+    <xacro:include filename="$(find phantomx_pincher_arm_description)/urdf/phantomx_pincher_arm.xacro"/>
 </robot>

Commit message: updates to enable multiple robots and scanse sensor

File: src/turtlebot2i/turtlebot2i_description/robots/kobuki_interbotix_astra.urdf.xacro (robot description, xacro)
@@ -12,7 +12,28 @@
   <sensor_astra parent="base_link"/>
   <sensor_sr300 parent="base_link"/>
+  <!--<sensor_scanse parent="base_link"/>-->
   <phantomx_pincher_arm parent="base_link" color="Red" gripper_color="Red">
     <!--<origin xyz="0.145 0.0 0.112"/>-->
     <origin xyz="0.145 0.0 0.148"/>
   </phantomx_pincher_arm>
+  <joint name="scanse_lidar_joint" type="fixed">
+    <origin xyz="0 0 0.485"
+            rpy="0 0 0"/>
+    <parent link="base_link"/>
+    <child link="lidar/scan" />
+  </joint>
+  <link name="lidar/scan">
+    <visual>
+      <origin xyz="0 0 0" rpy="0 0 0"/>
+      <geometry>
+        <cylinder length="0.0619" radius="0.0325"/>
+      </geometry>
+      <material name="blue"/>
+    </visual>
+    <collision>
+      <geometry>
+        <cylinder length="0.619" radius="0.325"/>
+      </geometry>
+    </collision>
+  </link>
 </robot>

File: src/turtlebot2i/turtlebot2i_description/urdf/turtlebot_library.urdf.xacro (robot description, xacro)
@@ -15,4 +15,5 @@
   <xacro:include filename="$(find turtlebot2i_description)/urdf/sensors/sr300.urdf.xacro"/>
   <xacro:include filename="$(find turtlebot2i_description)/urdf/sensors/zr300.urdf.xacro"/>
+  <xacro:include filename="$(find turtlebot2i_description)/urdf/sensors/scanse.urdf.xacro"/>
   <!-- Arms -->
   <xacro:include filename="$(find turtlebot2i_description)/urdf/arms/phantomx_pincher_arm.urdf.xacro"/>

Commit message: Fix typo on collision layer dimension

File: src/turtlebot2i/turtlebot2i_description/robots/kobuki_interbotix_astra.urdf.xacro (robot description, xacro)
@@ -33,5 +33,5 @@
     <collision>
       <geometry>
-        <cylinder length="0.619" radius="0.325"/>
+        <cylinder length="0.0619" radius="0.0325"/>
       </geometry>
     </collision>

Commit message: fixed lidar xacro and WH map parameters; added navigation script for single robot

File: src/turtlebot2i/turtlebot2i_description/robots/kobuki_interbotix_astra.urdf.xacro (robot description, xacro)
@@ -18,5 +18,7 @@
   </phantomx_pincher_arm>
   <joint name="scanse_lidar_joint" type="fixed">
-    <origin xyz="0 0 0.485"
+    <!--<origin xyz="0 0 0.485"
+            rpy="0 0 0"/>-->
+    <origin xyz="0.20 0 0.05"
             rpy="0 0 0"/>
     <parent link="base_link"/>
