Commit message: [backport] change upper limit when gripper is open

File: simulation-ros/src/phantomx_pincher_arm/phantomx_pincher_arm_description/urdf/phantomx_pincher_gripper.xacro (robot description, xacro)
@@ -7,5 +7,5 @@
       <origin xyz="0.070 0 0" rpy="0 0 0"/>
       <axis xyz="0 1 0"/>
-      <limit effort="30" velocity="0.5" lower="0.002" upper="0.032"/>
+      <limit effort="30" velocity="0.5" lower="0.002" upper="0.038"/>
       <parent link="arm_wrist_flex_link"/>
       <child link="gripper_active_link"/>
