Commit message: [backport] increase collision mesh size to improve collision checking

File: simulation-ros/src/phantomx_pincher_arm/phantomx_pincher_arm_description/urdf/arm_hardware.xacro (robot description, xacro)
@@ -205,5 +205,5 @@
         <xacro:insert_block name="origin"/>
         <geometry>
-          <mesh filename="package://phantomx_pincher_arm_description/meshes/PincherFinger.stl" scale="1.0 1.0 1.0"/>
+          <mesh filename="package://phantomx_pincher_arm_description/meshes/PincherFinger.stl" scale="1.05 1.05 1.05"/>
         </geometry>
       </collision>

Commit message: Increased gripper collision layer

File: simulation-ros/src/phantomx_pincher_arm/phantomx_pincher_arm_description/urdf/arm_hardware.xacro (robot description, xacro)
@@ -205,5 +205,5 @@
         <xacro:insert_block name="origin"/>
         <geometry>
-          <mesh filename="package://phantomx_pincher_arm_description/meshes/PincherFinger.stl" scale="1.05 1.05 1.05"/>
+          <mesh filename="package://phantomx_pincher_arm_description/meshes/PincherFinger.stl" scale="1.1 1.1 1.1"/>
         </geometry>
       </collision>

Commit message: Improved plan
- Improved successful rate on pick and drop tasks
- Reposition the robot to pick products

File: simulation-ros/src/phantomx_pincher_arm/phantomx_pincher_arm_description/urdf/arm_hardware.xacro (robot description, xacro)
@@ -205,5 +205,5 @@
         <xacro:insert_block name="origin"/>
         <geometry>
-          <mesh filename="package://phantomx_pincher_arm_description/meshes/PincherFinger.stl" scale="1.0 1.0 1.0"/>
+          <mesh filename="package://phantomx_pincher_arm_description/meshes/PincherFinger.stl" scale="1.1 1.1 1.1"/>
         </geometry>
       </collision>

File: simulation-ros/src/phantomx_pincher_arm/phantomx_pincher_arm_description/urdf/phantomx_pincher_arm.xacro (robot description, xacro)
@@ -73,5 +73,5 @@
     <link name="gripper_link"/>
     <joint name="PhantomXPincher_gripperCenter_joint" type="revolute">
-      <origin xyz="0.110 0 0" rpy="0 0 0"/>
+      <origin xyz="0.085 0 0" rpy="0 0 0"/>
       <parent link="arm_wrist_flex_link"/>
       <child link="gripper_link"/>

File: simulation-ros/src/turtlebot2i/turtlebot2i_description/robots/kobuki_interbotix_astra.urdf.xacro (robot description, xacro)
@@ -14,6 +14,6 @@
   <!--<sensor_scanse parent="base_link"/>-->
   <phantomx_pincher_arm parent="base_link" color="Red" gripper_color="Red">
-    <!--<origin xyz="0.145 0.0 0.112"/>-->
-    <origin xyz="0.145 0.0 0.148"/>
+    <origin xyz="0.145 0.0 0.112"/>
+    <!--<origin xyz="0.145 0.0 0.148"/>-->
   </phantomx_pincher_arm>
   <joint name="scanse_lidar_joint" type="fixed">

File: simulation-ros/src/turtlebot2i/turtlebot2i_description/urdf/arms/phantomx_pincher_arm.urdf.xacro (robot description, xacro)
@@ -4,5 +4,5 @@
     <!-- We can configure joints velocity limit and lower/upper limits
     to allow access to different operational areas, e.g. left handed vs. right handed robot -->
-    <xacro:property name="joints_vlimit" value="1.571"/>
+    <xacro:property name="joints_vlimit" value="0.571"/>
     <xacro:property name="pan_llimit" value="-3.1416"/>
     <xacro:property name="pan_ulimit" value="3.1416"/>
@@ -11,6 +11,6 @@
     <xacro:property name="elbow_llimit" value="-3.1416"/>
     <xacro:property name="elbow_ulimit" value="0.33516"/>
-    <xacro:property name="wrist_llimit" value="-1.57"/>
-    <xacro:property name="wrist_ulimit" value="1.57"/>
+    <xacro:property name="wrist_llimit" value="-1.55"/>
+    <xacro:property name="wrist_ulimit" value="1.55"/>
     <!-- We can configure joints velocity limit and lower/upper limits
     to allow access to different operational areas, e.g. left handed vs. right handed robot -->
