Commit message: Change joint limits to don't force position on v-rep

File: simulation-ros/src/turtlebot2i/turtlebot2i_description/urdf/arms/phantomx_pincher_arm.urdf.xacro (robot description, xacro)
@@ -11,6 +11,6 @@
     <xacro:property name="elbow_llimit" value="-3.1416"/>
     <xacro:property name="elbow_ulimit" value="0.33516"/>
-    <xacro:property name="wrist_llimit" value="-1.57"/>
-    <xacro:property name="wrist_ulimit" value="1.57"/>
+    <xacro:property name="wrist_llimit" value="-1.55"/>
+    <xacro:property name="wrist_ulimit" value="1.55"/>
     <!-- We can configure joints velocity limit and lower/upper limits
     to allow access to different operational areas, e.g. left handed vs. right handed robot -->

Commit message: Changed controllers parameters to cope with low FPS in V-REP
- Changed the gripper controller to FollowTrajectory as it's easier to add tolerances on execution
- Moveit will no longer track the time execution on the controllers
- Increased time scaling to move arm slower
- Changed the joint velocity upper limit to make it slower
- Changed the controller constraints to accomodate the delays from v-rep. Due to delays the arm controller is unable to follow the trajectory as close as it need so we increased all tolerances.

File: simulation-ros/src/turtlebot2i/turtlebot2i_description/urdf/arms/phantomx_pincher_arm.urdf.xacro (robot description, xacro)
@@ -4,5 +4,5 @@
     <!-- We can configure joints velocity limit and lower/upper limits
     to allow access to different operational areas, e.g. left handed vs. right handed robot -->
-    <xacro:property name="joints_vlimit" value="1.571"/>
+    <xacro:property name="joints_vlimit" value="0.571"/>
     <xacro:property name="pan_llimit" value="-3.1416"/>
     <xacro:property name="pan_ulimit" value="3.1416"/>
