Commit message: updated for 10x15m scenario

File: simulation-ros/src/turtlebot2i/turtlebot2i_description/robots/kobuki_interbotix_astra.urdf.xacro (robot description, xacro)
@@ -20,5 +20,5 @@
     <!--<origin xyz="0 0 0.485"
             rpy="0 0 0"/>-->
-    <origin xyz="0.20 0 0.05"
+    <origin xyz="0 0 0.5"
             rpy="0 0 0"/>
     <parent link="base_link"/>

Commit message: LIDAR moved to the base

File: simulation-ros/src/turtlebot2i/turtlebot2i_description/robots/kobuki_interbotix_astra.urdf.xacro (robot description, xacro)
@@ -20,5 +20,5 @@
     <!--<origin xyz="0 0 0.485"
             rpy="0 0 0"/>-->
-    <origin xyz="0 0 0.5"
+    <origin xyz="0.20 0 0.05"
             rpy="0 0 0"/>
     <parent link="base_link"/>

Commit message: demo preparation

File: simulation-ros/src/turtlebot2i/turtlebot2i_description/robots/kobuki_interbotix_astra.urdf.xacro (robot description, xacro)
@@ -18,8 +18,8 @@
   </phantomx_pincher_arm>
   <joint name="scanse_lidar_joint" type="fixed">
-    <!--<origin xyz="0 0 0.485"
+    <origin xyz="-0.05 0.001 0.485"
+            rpy="0 0 0"/>
+    <!--<origin xyz="0.20 0 0.05"
             rpy="0 0 0"/>-->
-    <origin xyz="0.20 0 0.05"
-            rpy="0 0 0"/>
     <parent link="base_link"/>
     <child link="lidar/scan" />
